Commit message: first commit

File: src/tri_steer_description/urdf/tri_steer.xacro (robot description, xacro)
@@ -557,5 +557,5 @@
     <child link="laser"/>
     <!-- 例：雷达在车体前方 0.20m，高 0.12m -->
-    <origin xyz="0.0 0 0.3" rpy="0 0 0"/>
+    <origin xyz="0.23 0.0 0.08" rpy="0 0 0"/>
     <!-- <origin xyz="0.0 0.5 0.0" rpy="0 0 0"/> -->
     <!-- <origin xyz="0.0 0.5 0.0" rpy="1.5708 0 0"/> -->
@@ -752,5 +752,5 @@
       <updateRate>100.0</updateRate>
       <bodyName>base_footprint</bodyName>
-      <topicName>carto_odom</topicName>
+      <topicName>odom</topicName>
       <gaussianNoise>0.0</gaussianNoise>
       <frameName>map</frameName>
